Commit message: update to xacro.load_yaml()

File: isuzu_sensor_description/urdf/sensor_kit.xacro (robot description, xacro)
@@ -17,5 +17,5 @@
     </link>
     <!-- sensor -->
-    <xacro:property name="calibration" value="${load_yaml('$(arg config_dir)/sensor_kit_calibration.yaml')}"/>
+    <xacro:property name="calibration" value="${xacro.load_yaml('$(arg config_dir)/sensor_kit_calibration.yaml')}"/>
     <!-- lidar -->
     <xacro:VLP-16 parent="sensor_kit_base_link" name="velodyne_front" topic="/velodyne_points" hz="10" samples="220" gpu="$(arg gpu)">

File: isuzu_sensor_description/urdf/sensors.xacro (robot description, xacro)
@@ -2,5 +2,5 @@
 <robot name="vehicle" xmlns:xacro="http://ros.org/wiki/xacro">
   <xacro:arg name="config_dir" default="$(find isuzu_sensor_description)/config"/>
-  <xacro:property name="calibration" value="${load_yaml('$(arg config_dir)/sensors_calibration.yaml')}"/>
+  <xacro:property name="calibration" value="${xacro.load_yaml('$(arg config_dir)/sensors_calibration.yaml')}"/>
   <!-- sensor kit -->
   <xacro:include filename="sensor_kit.xacro"/>
